Commit message: add d435

File: src/robots/go2_description/xacro/robot.xacro (robot description, xacro)
@@ -3,3 +3,7 @@
     <xacro:include filename="$(find go2_description)/urdf/go2_description.urdf"/>
     <xacro:include filename="$(find go2_description)/xacro/gazebo.xacro"/>
+    <xacro:include filename="$(find go2_description)/xacro/_d435i.urdf.xacro"/>
+    <xacro:sensor_d435i parent = "base" name = "camera" topics_ns="camera">
+        <origin xyz="0.345 0 0.07" rpy="0 0.25 0"/>
+    </xacro:sensor_d435i>
 </robot>
